File: kicad/kicad.kicad_pcb (KiCad board)
At the start: 2 copper layers, 57.8 x 85.7 mm, 78 parts, among them J1 USB_B, J2 Conn_02x03_Odd_Even, P1 POWER_IN, Q1 BSS84LT1, Q2 BSS84LT1, Q3 BC847, Q4 BC847, Q5 BC847, Q6 BSS84LT1, Q7 BSS84LT1, Q8 BSS84LT1, SW1 Reset, U1 74HC595, U2 74HC595, U3 MT3608, U4 ZIF28, U5 ATmega328P-A, U6 CH340C, U7 AMS1117-5.0, Y1 16MHz

Commit message: Small pre-release fixes
Parts:
- removed R7, R8: 4.7k, Resistor_SMD:R_0805_2012Metric_Pad1.20x1.40mm_HandSolder
- added REF**: MountingHole_2.7mm_M2.5, MountingHole:MountingHole_2.7mm_M2.5, F.Cu at (43.8, 37.5)
- added REF**: MountingHole_2.7mm_M2.5, MountingHole:MountingHole_2.7mm_M2.5, F.Cu at (90.2, 111.8)
- added REF**: MountingHole_2.7mm_M2.5, MountingHole:MountingHole_2.7mm_M2.5, F.Cu at (43.8, 111.8)
- added REF**: MountingHole_2.7mm_M2.5, MountingHole:MountingHole_2.7mm_M2.5, F.Cu at (90.2, 37.5)
- C12, C7: footprint Capacitor_Tantalum_SMD:CP_EIA-7361-38_AVX-V_Pad2.18x3.30mm_HandSolder -> Capacitor_Tantalum_SMD:CP_EIA-3216-18_Kemet-A_Pad1.58x1.35mm_HandSolder; moved to B.Cu
- C6, C8, R27, U6, U7: moved to B.Cu
- J2: footprint Connector_IDC:IDC-Header_2x03_P2.54mm_Vertical -> Connector_PinHeader_2.54mm:PinHeader_2x03_P2.54mm_Vertical
- R31: renamed from R26; moved to B.Cu
- SW1: footprint Button_Switch_SMD:Nidec_Copal_SH-7010A -> Button_Switch_SMD:SW_SPST_TL3342
- Y1: footprint Crystal:Resonator_SMD_Murata_CSTxExxV-3Pin_3.0x1.1mm_HandSoldering -> Crystal:Resonator_SMD_Murata_CSTxExxV-3Pin_3.0x1.1mm
- moved R31 71.5 mm to (54.0, 109.2), turned to 180 degrees
- moved C9 55.8 mm to (82.0, 62.4)
- moved R30 52.6 mm to (49.7, 97.8), turned to 180 degrees
- moved LED3 51.1 mm to (54.0, 97.8), turned to 180 degrees
- moved R29 49.2 mm to (49.7, 102.9), turned to 180 degrees
- moved P1 48.8 mm to (91.1, 99.1), turned to -90 degrees
- moved SW1 47.5 mm to (81.0, 109.3), turned to 90 degrees
- moved J2 46.7 mm to (63.0, 90.7), turned to -90 degrees
- moved LED2 46.4 mm to (54.0, 102.9), turned to 180 degrees
- moved R12 46.1 mm to (79.4, 88.5), turned to 90 degrees
- moved C11 43.2 mm to (49.7, 110.6)
- moved R10 42.7 mm to (40.6, 59.7)
- moved U7 40.6 mm to (83.8, 101.6), turned to 180 degrees
- moved R22 40.3 mm to (48.5, 56.6), turned to 0 degrees
- moved R27 38.7 mm to (57.1, 111.4)
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- renumbered D12 to LED2, D13 to LED3, R11 to R10, R12 to R11, R10 to R12, R19 to R20, R20 to R21, R21 to R22, R22 to R23, R23 to R24, R24 to R25, R25 to R26
Connections:
- net /EPROM27/NEXT_1 renamed NEXT_1
- net Net-(D11-A) renamed /Arduino/+5_USB
- net RESET renamed A6_IN
- C6 pad 1: VCC -> +5V
- C7 pad 1: VCC -> +5V
- C9 pad 1: VCC -> +5V
- D11 pad 1: VCC -> +5V
- D2 pad 2: Net-(A2-A7) -> ADC
- D3 pad 2: Net-(A2-A4/SDA) -> SDA
- J1 pad 5: unconnected-(J1-Shield-Pad5) -> GND
- J1 pad 6: (no net) -> GND
- J2 pad 2: VCC -> +5V
- R1 pad 1: /EPROM27/R_A11 -> MISO
- R10 pad 1: /EPROM27/E_A15 -> E_A15
- R11 pad 1: /EPROM27/E_A11 -> E_A11
- R12 pad 1: /EPROM27/E_OE -> E_OE
- R13 pad 1: GND -> Net-(Q3-E)
- R13 pad 2: Net-(Q3-E) -> GND
- R14 pad 1: GND -> Net-(Q4-E)
- R14 pad 2: Net-(Q4-E) -> GND
- R15 pad 1: GND -> Net-(Q5-E)
- R15 pad 2: Net-(Q5-E) -> GND
- R2 pad 1: /EPROM27/R_A13 -> R_A13
- R28 pad 2: VCC -> +5V
- R29 pad 2: VCC -> +5V
- R30 pad 2: VCC -> +5V
- R6 pad 2: Net-(A2-A7) -> ADC
- R9 pad 1: Net-(A2-A7) -> ADC
- U1 pad 10: /EPROM27/SS -> +5V
- U1 pad 11: /EPROM27/SCK -> SCK
- U1 pad 12: +5V -> SS
- U1 pad 14: /EPROM27/MOSI -> MOSI
- U2 pad 10: /EPROM27/SS -> +5V
- U2 pad 11: /EPROM27/SCK -> SCK
- U2 pad 12: +5V -> SS
- U3 pad 4: unconnected-(U3-EN-Pad4) -> +5V
- U3 pad 5: unconnected-(U3-IN-Pad5) -> +5V
- U4 pad 11: /EPROM27/D0 -> D0
- U4 pad 12: /EPROM27/D1 -> D1
- U4 pad 13: /EPROM27/D2 -> D2
- U4 pad 15: /EPROM27/D3 -> D3
- U4 pad 16: /EPROM27/D4 -> D4
- U4 pad 17: /EPROM27/D5 -> D5
- U4 pad 18: /EPROM27/D6 -> D6
- U4 pad 19: /EPROM27/D7 -> D7
- U4 pad 20: /EPROM27/CE -> CE
- U5 pad 1: unconnected-(U5-PD3-Pad1) -> D1
- U5 pad 10: unconnected-(U5-PD6-Pad10) -> D4
- U5 pad 11: unconnected-(U5-PD7-Pad11) -> D5
- U5 pad 12: unconnected-(U5-PB0-Pad12) -> D6
- U5 pad 13: unconnected-(U5-PB1-Pad13) -> D7
- U5 pad 14: unconnected-(U5-PB2-Pad14) -> SS
- U5 pad 18: VCC -> +5V
- U5 pad 2: unconnected-(U5-PD4-Pad2) -> D2
- U5 pad 22: unconnected-(U5-ADC7-Pad22) -> ADC
- U5 pad 23: unconnected-(U5-PC0-Pad23) -> E_OE
- U5 pad 24: unconnected-(U5-PC1-Pad24) -> E_A15
- U5 pad 25: unconnected-(U5-PC2-Pad25) -> E_A11
- U5 pad 26: unconnected-(U5-PC3-Pad26) -> CE
- U5 pad 27: unconnected-(U5-PC4-Pad27) -> SDA
- U5 pad 28: unconnected-(U5-PC5-Pad28) -> R_A13
- U5 pad 32: unconnected-(U5-PD2-Pad32) -> D0
- U5 pad 4: VCC -> +5V
- U5 pad 6: VCC -> +5V
- U5 pad 9: unconnected-(U5-PD5-Pad9) -> D3
- U6 pad 16: VCC -> +5V
- U7 pad 2: VCC -> +5V
Routing:
- net +5V: track 0.00 -> 250.6 mm, vias 0 -> 8
- net VCC: track 0.00 -> 207.6 mm
- net SCK: track 0.00 -> 81.1 mm, vias 0 -> 2
- net MOSI: track 0.00 -> 67.8 mm, vias 0 -> 1
- net SS: track 0.00 -> 65.6 mm
- net E_A15: track 0.00 -> 62.2 mm, vias 0 -> 2
- net D0: track 0.00 -> 59.4 mm, vias 0 -> 2
- net A6_IN: track 0.00 -> 55.3 mm, vias 0 -> 1
- net R_A13: track 0.00 -> 53.1 mm, vias 0 -> 2
- net /EPROM27/A8: track 0.00 -> 52.0 mm, vias 0 -> 2
- net SDA: track 0.00 -> 51.2 mm, vias 0 -> 3
- net CE: track 0.00 -> 48.1 mm, vias 0 -> 1
- net /EPROM27/A14: track 0.00 -> 44.8 mm, vias 0 -> 1
- net D1: track 0.00 -> 43.2 mm, vias 0 -> 2
- net /EPROM27/A9: track 0.00 -> 42.9 mm, vias 0 -> 3
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- added copper zone on B.Cu, net GND
- added copper zone on F.Cu, net GND
Other:
- outline, holes or cut-outs redrawn
- board text added: "EPROM 27 PROGRAMMER rev. 3.0"
- board text added: "RX"
- board text added: "TX"
- board text added: "github.com/ walhi Radionews kab01m"
