File: kicad/kicad.kicad_sch (KiCad schematic)
At the start: 0 parts

Commit message: Small pre-release fixes
Other:
- company: (none) -> kab01m@github
- title: (none) -> EPROM27 Arduino programmer
Changed lines of the file:
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@@
 	(generator "eeschema")
 	(generator_version "8.0")
-	(paper "User" 292.1 205.105)
+	(paper "A2")
+	(title_block
+		(title "EPROM27 Arduino programmer")
+		(date "2024-03-21")
+		(rev "3.0")
+		(company "kab01m@github")
+	)
 	(sheet
-		(at 0 -382.27)
-		(size 290.83 173.99)
+		(at 308.61 171.45)
+		(size 269.24 198.12)
 		(fields_autoplaced yes)
 		(stroke
@@
 		)
 		(property "Sheetname" "EPROM27"
-			(at 0 -382.9816 0)
+			(at 308.61 170.7384 0)
 			(effects
 				(font
@@
 		)
 		(property "Sheetfile" "eprom27.kicad_sch"
-			(at 0 -207.6954 0)
-			(effects
-				(font
-					(size 1.27 1.27)
-				)
-				(justify left top)
-			)
-		)
-		(instances
-			(project "kicad"
-				(path "/b8033ce9-ba25-4e47-95e8-10bc4b45a8e3"
-					(page "1")
-				)
-			)
-		)
-	)
-	(sheet
-		(at 0 -196.85)
-		(size 290.83 189.23)
-		(fields_autoplaced yes)
-		(stroke
-			(width 0.1524)
-			(type solid)
-		)
-		(fill
-			(color 0 0 0 0.0000)
-		)
-		(property "Sheetname" "Arduino"
-			(at 0 -197.5616 0)
-			(effects
-				(font
-					(size 1.27 1.27)
-				)
-				(justify left bottom)
-			)
-		)
-		(property "Sheetfile" "arduino.kicad_sch"
-			(at 0 -7.0354 0)
+			(at 308.61 370.1546 0)
 			(effects
 				(font
@@
 		)
 	)
+	(sheet
+		(at 24.13 16.51)
+		(size 275.59 190.5)
+		(fields_autoplaced yes)
+		(stroke
+			(width 0.1524)
+			(type solid)
+		)
+		(fill
+			(color 0 0 0 0.0000)
+		)
+		(property "Sheetname" "Arduino"
+			(at 24.13 15.7984 0)
+			(effects
+				(font
+					(size 1.27 1.27)
+				)
+				(justify left bottom)
+			)
+		)
+		(property "Sheetfile" "arduino.kicad_sch"
+			(at 24.13 207.5946 0)
+			(effects
+				(font
+					(size 1.27 1.27)
+				)
+				(justify left top)
+			)
+		)
+		(instances
+			(project "kicad"
+				(path "/b8033ce9-ba25-4e47-95e8-10bc4b45a8e3"
+					(page "3")
+				)
+			)
+		)
+	)
 	(sheet_instances
 		(path "/"
-			(page "0")
+			(page "1")
 		)
 	)
